Commit message: UPdate scale since STL is in mm but ROS takes them as meters

File: hopper_description/urdf/hopper.urdf (robot description, URDF)
Before this commit: robot Hopper, 1 links, 0 joints
Links:
- link base_link: geometry visual mesh filename=package://hopper_description/meshes/hopper_body.stl scale=0.001 0.001 0.001

Commit message: Fix orientation in udrf files

File: hopper_description/urdf/hopper.urdf (robot description, URDF)
Before this commit: robot Hopper, 3 links, 2 joints
Joints:
- joint base_to_left_front_coxa: origin xyz=0.115 0.05 0.0 rpy=0.0 0.0 0.0 -> xyz=-0.05 0.115 0.0 rpy=0.0 0.0 0.0
- joint base_to_right_front_coxa: origin xyz=0.115 0.05 0.0 rpy=0.0 0.0 0.0 -> xyz=0.05 0.115 0.0 rpy=0.0 0.0 0.0

Commit message: Add simple urdf description

File: hopper_description/urdf/hopper.urdf (robot description, URDF)
Before this commit: robot Hopper, 1 links, 0 joints
Links:
- added link left_front_coxa; visual mesh filename=package://hopper_description/meshes/hopper_leg_coxa.stl scale=0.001 0.001 0.001
- added link right_front_coxa; visual mesh filename=package://hopper_description/meshes/hopper_leg_coxa.stl scale=0.001 0.001 0.001
Joints:
- added joint base_to_left_front_coxa: type fixed, parent base_link, child left_front_coxa, origin xyz=0.115 0.05 0.0 rpy=0.0 0.0 0.0, axis 0.0 0.0 0.0
- added joint base_to_right_front_coxa: type fixed, parent base_link, child right_front_coxa, origin xyz=0.115 0.05 0.0 rpy=0.0 0.0 0.0, axis 0.0 0.0 0.0
