Commit message: Fix repeated typo in word xacro

File: hopper_description/urdf/hopper.xacro (robot description, xacro)
@@ -2,6 +2,6 @@
 <robot
     xmlns:xacro="http://ros.org/wiki/xacro" name="Hopper">
-    <xacro:property name="coxa_length" value="0.05" />
-    <xacro:property name="femur_length" value="0.067" />
+    <xacro:property name="coxa_length" value="0.044" />
+    <xacro:property name="femur_length" value="0.07" />
     <material name="white">
         <color rgba="1 1 1 1"/>
@@ -50,4 +50,11 @@
         <origin xyz="0.025 0 0.11" rpy="0 0 ${pi}"/>
     </joint>
+    <!-- IMU attachment -->
+    <link name="imu"/>
+    <joint name="body_imu_joint" type="fixed">
+        <parent link="body_link" />
+        <child link="imu" />
+        <origin xyz="0.025 0 0" rpy="0 0 ${pi}"/>
+    </joint>
     <!-- Stereo camera  -->
     <link name="stereo_camera"/>
@@ -69,5 +76,5 @@
         <origin xyz="0 -0.07 0" rpy="0 ${pi/2} 0" />
     </joint>
-    <!-- xarco macro for leg -->
+    <!-- xacro macro for leg -->
     <xacro:macro name="leg" params="side position x y angle axis">
         <!-- leg base -->
@@ -128,9 +135,9 @@
     </xacro:macro>
     <!--build legs-->
-    <xacro:leg side="right" position="rear" x="-0.115" y="-0.050" angle="-${pi*3/4}" axis="1" />
-    <xacro:leg side="right" position="middle" x="0.0" y="-0.100" angle="-${pi/2}" axis="1" />
-    <xacro:leg side="right" position="front" x="0.115" y="-0.050" angle="-${pi/4}" axis="1" />
-    <xacro:leg side="left" position="rear" x="-0.115" y="0.050" angle="${pi*3/4}" axis="-1" />
-    <xacro:leg side="left" position="middle" x="0.0" y="0.100" angle="${pi/2}" axis="-1" />
-    <xacro:leg side="left" position="front" x="0.115" y="0.050" angle="${pi/4}" axis="-1" />
+    <xacro:leg side="right" position="rear" x="-0.115" y="-0.063" angle="-${pi/2}" axis="1" />
+    <xacro:leg side="right" position="middle" x="0.0" y="-0.103" angle="-${pi/2}" axis="1" />
+    <xacro:leg side="right" position="front" x="0.115" y="-0.063" angle="-${pi/2}" axis="1" />
+    <xacro:leg side="left" position="rear" x="-0.115" y="0.063" angle="${pi/2}" axis="-1" />
+    <xacro:leg side="left" position="middle" x="0.0" y="0.103" angle="${pi/2}" axis="-1" />
+    <xacro:leg side="left" position="front" x="0.115" y="0.063" angle="${pi/2}" axis="-1" />
 </robot>

File: hopper_description/urdf/old_hopper.xacro (robot description, xacro)
@@ -2,6 +2,6 @@
 <robot
     xmlns:xacro="http://ros.org/wiki/xacro" name="Hopper">
-    <xacro:property name="coxa_length" value="0.044" />
-    <xacro:property name="femur_length" value="0.07" />
+    <xacro:property name="coxa_length" value="0.05" />
+    <xacro:property name="femur_length" value="0.067" />
     <material name="white">
         <color rgba="1 1 1 1"/>
@@ -50,11 +50,4 @@
         <origin xyz="0.025 0 0.11" rpy="0 0 ${pi}"/>
     </joint>
-    <!-- IMU attachment -->
-    <link name="imu"/>
-    <joint name="body_imu_joint" type="fixed">
-        <parent link="body_link" />
-        <child link="imu" />
-        <origin xyz="0.025 0 0" rpy="0 0 ${pi}"/>
-    </joint>
     <!-- Stereo camera  -->
     <link name="stereo_camera"/>
@@ -76,5 +69,5 @@
         <origin xyz="0 -0.07 0" rpy="0 ${pi/2} 0" />
     </joint>
-    <!-- xarco macro for leg -->
+    <!-- xacro macro for leg -->
     <xacro:macro name="leg" params="side position x y angle axis">
         <!-- leg base -->
@@ -135,9 +128,9 @@
     </xacro:macro>
     <!--build legs-->
-    <xacro:leg side="right" position="rear" x="-0.115" y="-0.063" angle="-${pi/2}" axis="1" />
-    <xacro:leg side="right" position="middle" x="0.0" y="-0.103" angle="-${pi/2}" axis="1" />
-    <xacro:leg side="right" position="front" x="0.115" y="-0.063" angle="-${pi/2}" axis="1" />
-    <xacro:leg side="left" position="rear" x="-0.115" y="0.063" angle="${pi/2}" axis="-1" />
-    <xacro:leg side="left" position="middle" x="0.0" y="0.103" angle="${pi/2}" axis="-1" />
-    <xacro:leg side="left" position="front" x="0.115" y="0.063" angle="${pi/2}" axis="-1" />
+    <xacro:leg side="right" position="rear" x="-0.115" y="-0.050" angle="-${pi*3/4}" axis="1" />
+    <xacro:leg side="right" position="middle" x="0.0" y="-0.100" angle="-${pi/2}" axis="1" />
+    <xacro:leg side="right" position="front" x="0.115" y="-0.050" angle="-${pi/4}" axis="1" />
+    <xacro:leg side="left" position="rear" x="-0.115" y="0.050" angle="${pi*3/4}" axis="-1" />
+    <xacro:leg side="left" position="middle" x="0.0" y="0.100" angle="${pi/2}" axis="-1" />
+    <xacro:leg side="left" position="front" x="0.115" y="0.050" angle="${pi/4}" axis="-1" />
 </robot>

Commit message: Update orientation of IMU

File: hopper_description/urdf/hopper.xacro (robot description, xacro)
@@ -55,5 +55,5 @@
         <parent link="body_link" />
         <child link="imu" />
-        <origin xyz="0.025 0 0" rpy="0 0 ${pi}"/>
+        <origin xyz="0.025 0 0" rpy="${pi} 0 ${pi}"/>
     </joint>
     <!-- Stereo camera  -->

Commit message: Publisher imu orientation

File: hopper_description/urdf/hopper.xacro (robot description, xacro)
@@ -24,9 +24,9 @@
         <child link="body_link" />
     </joint>
-    <link name="base_stabilized"/>
+    <!-- <link name="base_stabilized"/>
     <joint name="base_orientation_joint" type="fixed">
         <parent link="base_stabilized" />
         <child link="base_link" />
-    </joint>
+    </joint> -->
     <!-- forward arrow -->
     <link name="arrow">

Commit message: Add tf link for feet sensor

File: hopper_description/urdf/hopper.xacro (robot description, xacro)
@@ -4,4 +4,5 @@
     <xacro:property name="coxa_length" value="0.044" />
     <xacro:property name="femur_length" value="0.07" />
+    <xacro:property name="tibia_length" value="0.128" />
     <material name="white">
         <color rgba="1 1 1 1"/>
@@ -133,4 +134,10 @@
             <limit lower="-${pi}" upper="${pi}" effort="1000.0" velocity="1"/>
         </joint>
+        <link name="${side}_${position}_button"/>
+        <joint name="${side}_${position}_tibia_button" type="fixed">
+            <origin xyz="${tibia_length} 0.0 0.0"/>
+            <parent link="${side}_${position}_tibia" />
+            <child link="${side}_${position}_button" />
+        </joint>
     </xacro:macro>
     <!--build legs-->

Commit message: Fix lidar position

File: hopper_description/urdf/hopper.xacro (robot description, xacro)
@@ -49,5 +49,5 @@
         <parent link="body_link" />
         <child link="laser" />
-        <origin xyz="0.025 0 0.11" rpy="0 0 ${pi}"/>
+        <origin xyz="0.035 0 0.112" rpy="0 0 ${pi}"/>
     </joint>
     <!-- IMU attachment -->
@@ -59,5 +59,5 @@
     </joint>
     <!-- Stereo camera  -->
-    <link name="stereo_camera"/>
+    <!-- <link name="stereo_camera"/>
     <joint name="body_camera_joint" type="fixed">
         <parent link="body_link" />
@@ -76,5 +76,5 @@
         <child link="right_camera" />
         <origin xyz="0 -0.07 0" rpy="0 ${pi/2} 0" />
-    </joint>
+    </joint> -->
     <!-- xacro macro for leg -->
     <xacro:macro name="leg" params="side position x y angle axis">

Commit message: Update urdf to use model with lidar and shrink size of axes in rviz

File: hopper_description/urdf/hopper.xacro (robot description, xacro)
@@ -16,5 +16,5 @@
         <visual>
             <geometry>
-                <mesh filename="package://hopper_description/meshes/hopper_body.stl" scale="0.001 0.001 0.001"/>
+                <mesh filename="package://hopper_description/meshes/hopper_body_full.stl" scale="0.001 0.001 0.001"/>
             </geometry>
             <material name="white"/>
